File: docs/kicad/adefesio.kicad_pcb (KiCad board)
At the start: 2 copper layers, 12 parts, among them J1 CONN_01X08, U1 ULN2003

Commit message: 2019-02-19 Procastinando
Parts:
- removed J1: CONN_01X08, Connectors_Samtec:SL-108-X-XX_1x08
- added A1: Arduino_Nano, arduino_nano:arduino_nano, F.Cu at (174.0, 143.5)
- added J2: MOTOR_IZQ, Connectors:PINHEAD1-6, F.Cu at (194.3, 94.0)
- added J3: MOTOR_DER, Connectors:PINHEAD1-6, F.Cu at (168.9, 92.7)
- added J4: CONN_01X02, Connectors:PINHEAD1-2, F.Cu at (222.2, 134.6)
- added R3: R, Resistors_THT:R_Axial_DIN0204_L3.6mm_D1.6mm_P7.62mm_Horizontal, F.Cu at (168.9, 141.0)
- added R4: R, Resistors_THT:R_Axial_DIN0204_L3.6mm_D1.6mm_P7.62mm_Horizontal, F.Cu at (176.5, 141.0)
- added SW1: SW_SPST, Buttons_Switches_SMD:SW_DIP_x1_W7.62mm_Slide_Copal_CHS-B, F.Cu at (226.1, 146.1)
- added U2: TB6612FNG_BREAKOUT, bl_kicad:DIP-16_600, F.Cu at (217.2, 135.9)
- moved D5 109.3 mm to (218.4, 83.8)
- moved D6 108.0 mm to (226.1, 83.8)
- moved D8 103.8 mm to (194.3, 59.7)
- moved D2 103.8 mm to (185.4, 59.7)
- moved D4 103.7 mm to (194.3, 67.3)
- moved D3 103.7 mm to (185.4, 67.3)
- moved U1 103.4 mm to (182.9, 85.1)
- moved R2 103.3 mm to (176.5, 71.1)
- moved R1 103.2 mm to (190.5, 69.8)
- moved D7 99.1 mm to (154.9, 83.8)
- moved D1 97.9 mm to (162.6, 83.8)
Routing:
- net GND: track 173.9 -> 0.00 mm
- net SENSOR: track 119.3 -> 0.00 mm
- net Net-(D1-Pad2): track 83.3 -> 0.00 mm
- net MOTOR_B2: track 0.00 -> 52.6 mm
- net MOTOR_B1: track 0.00 -> 52.6 mm
- net MOTOR_A1: track 0.00 -> 47.2 mm
- net MOTOR_A2: track 0.00 -> 47.2 mm
- net ENCODER_RIGHT_C2: track 0.00 -> 46.3 mm
- net Net-(D1-Pad1): track 45.3 -> 0.00 mm
- net ENCODER_RIGHT_C1: track 0.00 -> 44.2 mm
- net +5V: track 24.4 -> 0.00 mm
- net Net-(D5-Pad1): track 19.5 -> 0.00 mm
- net Net-(D3-Pad1): track 18.3 -> 0.00 mm
- net Net-(D4-Pad1): track 13.2 -> 0.00 mm
- net LED_IZQ: track 3.81 -> 0.00 mm
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