File: docs/kicad/adefesio.sch (KiCad schematic (older format))
At the start: 12 parts, among them J1 CONN_01X08, U1 ULN2003

Commit message: 2019-02-19 Procastinando
Parts:
- removed J1: CONN_01X08, Connectors_Samtec:SL-108-X-XX_1x08, symbol CONN_01X08
- added A1: Arduino_Nano, arduino_nano:arduino_nano, symbol Arduino_Nano
- added J2: MOTOR_IZQ, Connectors:PINHEAD1-6, symbol CONN_01X06
- added J3: MOTOR_DER, Connectors:PINHEAD1-6, symbol CONN_01X06
- added J4: CONN_01X02, Connectors:PINHEAD1-2, symbol CONN_01X02
- added R3, R4: R, Resistors_THT:R_Axial_DIN0204_L3.6mm_D1.6mm_P7.62mm_Horizontal, symbol R
- added SW1: SW_SPST, Buttons_Switches_SMD:SW_DIP_x1_W7.62mm_Slide_Copal_CHS-B, symbol SW_SPST
- added U2: TB6612FNG_BREAKOUT, bl_kicad:DIP-16_600, symbol TB6612FNG_BREAKOUT
Connections:
- net GND: now also A1.29 (GND), A1.4 (GND), J2.6 (P6), J3.1 (P1), J4.1 (P1), R4.2, U2.3 (GND), U2.8 (GND), U2.9 (GND)
- net LED_DER: now also A1.21 (AD2/D16)
- net LED_FDER: now also A1.23 (AD4/D18)
- net LED_FIZQ: now also A1.22 (AD3/D17)
- net LED_IZQ: now also A1.20 (AD1/D15)
- new net: J4.2 (P2), SW1.1 (A)
- new net 5V: A1.27 (5V), J2.5 (P5), J3.2 (P2), U2.13 (STBY), U2.2 (VCC)
- new net BATERIA_LED_PIN: A1.16 (D13)
- new net BATERIA_VOLTAJE_PIN: A1.19 (AD0/D14), R3.2, R4.1
- new net BLUETOOTH_RX: A1.2 (D0/TX)
- new net BLUETOOTH_TX: A1.1 (D1/RX)
- new net ENCODER_LEFT_C1: A1.5 (D2), J2.4 (P4)
- new net ENCODER_LEFT_C2: A1.15 (D12), J2.3 (P3)
- new net ENCODER_RIGHT_C1: A1.6 (D3), J3.4 (P4)
- new net ENCODER_RIGHT_C2: A1.11 (D8), J3.3 (P3)
- new net LED_SENSOR: A1.24 (AD5/D19)
- new net MOTOR_A1: J2.2 (P2), U2.4 (AO1)
- new net MOTOR_A2: J2.1 (P1), U2.5 (AO2)
- new net MOTOR_B1: J3.6 (P6), U2.6 (BO2)
- new net MOTOR_B2: J3.5 (P5), U2.7 (BO1)
- new net MOTOR_LEFT_IN1: A1.12 (D9), U2.15 (AIN2)
- new net MOTOR_LEFT_IN2: A1.7 (D4), U2.14 (AIN1)
- new net MOTOR_LEFT_PWM: A1.8 (D5), U2.16 (PWMA)
- new net MOTOR_RIGHT_IN1: A1.10 (D7), U2.11 (BIN2)
- new net MOTOR_RIGHT_IN2: A1.13 (D10), U2.12 (BIN1)
- new net MOTOR_RIGHT_PWM: A1.9 (D6), U2.10 (PWMB)
- new net VBAT: A1.30 (Vin), R3.1, SW1.2 (B), U2.1 (VMOT)
- no-connect marks 0 -> 3
